Commit message: added the robot model for the tracked robot and a diffdrive robot. Also, added ros2_control

File: ika_robot_description/test_robot_urdf/robot.xacro (robot description, xacro)
@@ -2,5 +2,4 @@
 <robot name="my_robot" xmlns:xacro="http://www.ros.org/wiki/xacro">
     <xacro:arg name="use_ros2_control" default="true"/>
-    <xacro:include filename="common_properties.xacro" />
     <xacro:include filename="robot_base.xacro"/>
     <xacro:if value="$(arg use_ros2_control)">

File: ika_robot_description/urdf/robot_base.xacro (robot description, xacro)
@@ -1,26 +1,130 @@
 <?xml version="1.0"?>
 <robot xmlns:xacro="http://www.ros.org/wiki/xacro">
-    <xacro:property name="base_length" value="1."/>
-    <xacro:property name="base_width" value=".6"/>
-    <xacro:property name="base_hight" value=".4"/>
-    <link name="base_footprint"></link>
+    <xacro:property name="base_length" value="1.2"/>
+    <xacro:property name="base_width" value="0.7"/>
+    <xacro:property name="base_hight" value=".2"/>
+    <xacro:property name="base_mass" value="30."/>
+    <xacro:property name="wheel_radius" value="0.3"/>
+    <xacro:property name="wheel_length" value="0.3"/>
+    <xacro:property name="wheel_mass" value="5."/>
+    <xacro:property name="wheel_number" value="5"/>
+    <xacro:property name="base_to_ground" value="${2*wheel_radius}"/>
+    <link name="base_footprint"/>
     <joint name="base_joint" type="fixed">
         <parent link="base_footprint"/>
         <child link="base_link"/>
-        <origin xyz="0 0 0.6" rpy="0 0 0"/>
+        <origin xyz="0 0 ${base_to_ground}"/>
     </joint>
+    <!-- Base Link -->
     <link name="base_link">
         <visual>
             <geometry>
-                <box size="${base_length} ${base_width} ${base_hight}"/>
+                <box size="${base_length} ${base_width} ${base_hight}" />
             </geometry>
-            <origin xyz="0 0 ${base_hight/2}"/>
+            <origin xyz="0 0 ${base_hight/2.}" rpy="0 0 0" />
+            <material name="green" />
         </visual>
         <collision>
             <geometry>
-                <box size="${base_length} ${base_width} ${base_hight}"/>
+                <box size="${base_length} ${base_width} ${base_hight}" />
             </geometry>
-            <origin xyz="0 0 ${base_hight/2}"/>
+            <origin xyz="0 0 ${base_hight/2.}" rpy="0 0 0" />
         </collision>
+        <xacro:box_inertia m="${base_mass}" l="${base_length}" w="${base_width}" h="${base_hight}"
+                           xyz="0 0 ${base_hight/2.}" rpy="0 0 0" />
     </link>
+    <!-- Left Wheels -->
+    <xacro:macro name="left_wheel" params="id">
+        <link name="left_wheel_${id}">
+            <visual>
+                <geometry>
+                    <cylinder radius="${wheel_radius}" length="${wheel_length}"/>
+                </geometry>
+                <material name="blue"/>
+            </visual>
+            <collision>
+                <geometry>
+                    <sphere radius="${wheel_radius}"/>
+                    <!-- <cylinder radius="${wheel_radius}" length="${wheel_length}"/> -->
+                </geometry>
+            </collision>
+            <xacro:cylinder_inertia m="${wheel_mass}" r="${wheel_length}" l = "${wheel_length}"
+                                    xyz="0 0 0" rpy="0 0 0"/>
+        </link>
+        <joint name="left_wheel_joint_${id}" type="continuous">
+            <parent link="base_link"/>
+            <child link="left_wheel_${id}"/>
+            <origin xyz="${base_length*(id-1)/(wheel_number-1) - base_length/2}
+                         ${base_width/2 + wheel_length/2} ${-wheel_radius}" rpy="${-pi/2.} 0 0"/>
+            <axis xyz="0 0 1"/>
+        </joint>
+    </xacro:macro>
+    <xacro:left_wheel id="1"/>
+    <xacro:left_wheel id="2"/>
+    <xacro:left_wheel id="3"/>
+    <xacro:left_wheel id="4"/>
+    <xacro:left_wheel id="5"/>
+    <!-- Right Wheels -->
+    <xacro:macro name="right_wheel" params="id">
+        <link name="right_wheel_${id}">
+            <visual>
+                <geometry>
+                    <cylinder radius="${wheel_radius}" length="${wheel_length}"/>
+                </geometry>
+                <material name="blue" />
+            </visual>
+            <collision>
+                <geometry>
+                    <sphere radius="${wheel_radius}"/>
+                    <!-- <cylinder radius="${wheel_radius}" length="${wheel_length}"/> -->
+                </geometry>
+            </collision>
+            <xacro:cylinder_inertia m="${wheel_mass}" r="${wheel_length}" l = "${wheel_length}"
+                                    xyz="0 0 0" rpy="0 0 0"/>
+        </link>
+        <joint name="right_wheel_joint_${id}" type="continuous">
+            <parent link="base_link"/>
+            <child link="right_wheel_${id}"/>
+            <origin xyz="${base_length*(id-1)/(wheel_number-1) - base_length/2}
+                         -${base_width/2 + wheel_length/2} ${-wheel_radius}" rpy="${pi/2.} 0 0"/>
+            <axis xyz="0 0 -1"/>
+        </joint>
+    </xacro:macro>
+    <xacro:right_wheel id="1"/>
+    <xacro:right_wheel id="2"/>
+    <xacro:right_wheel id="3"/>
+    <xacro:right_wheel id="4"/>
+    <xacro:right_wheel id="5"/>
+    <xacro:macro name="create_gazebo_mu_001_wheel_tag" params="link_name color">
+        <gazebo reference="${link_name}">
+            <material>Gazebo/${color}</material>
+            <mu1 value="0.001"></mu1>
+            <mu2 value="0.001"></mu2>
+        </gazebo>
+    </xacro:macro>
+    <xacro:macro name="create_gazebo_mu_05_wheel_tag" params="link_name color">
+        <gazebo reference="${link_name}">
+            <material>Gazebo/${color}</material>
+            <mu1 value="0.05"></mu1>
+            <mu2 value="0.05"></mu2>
+        </gazebo>
+    </xacro:macro>
+    <xacro:create_gazebo_mu_001_wheel_tag link_name="left_wheel_1" color="Yellow"/>
+    <xacro:create_gazebo_mu_001_wheel_tag link_name="right_wheel_1" color="Orange"/>
+    <xacro:create_gazebo_mu_05_wheel_tag link_name="left_wheel_2" color="Yellow"/>
+    <xacro:create_gazebo_mu_05_wheel_tag link_name="right_wheel_2" color="Orange"/>
+    <xacro:create_gazebo_mu_05_wheel_tag link_name="left_wheel_4" color="Yellow"/>
+    <xacro:create_gazebo_mu_05_wheel_tag link_name="right_wheel_4" color="Orange"/>
+    <xacro:create_gazebo_mu_001_wheel_tag link_name="left_wheel_5" color="Yellow"/>
+    <xacro:create_gazebo_mu_001_wheel_tag link_name="right_wheel_5" color="Orange"/>
+    <gazebo reference="left_wheel_3">
+        <material>Gazebo/Yellow</material>
+        <mu1 value="1"></mu1>
+        <mu2 value="1"></mu2>
+    </gazebo>
+    <gazebo reference="right_wheel_3">
+        <material>Gazebo/Orange</material>
+        <mu1 value="1"></mu1>
+        <mu2 value="1"></mu2>
+    </gazebo>
 </robot>
