Commit message: added enable_track and section1

File: ika_robot_description/urdf/common_properties.xacro (robot description, xacro)
@@ -12,4 +12,7 @@
     <material name="orange">
         <color rgba="1 0.3 0 1"/>
+    </material>
+    <material name="yellow">
+        <color rgba="1 1 0 1"/>
     </material>
     <xacro:macro name="sphere_inertia" params="m r xyz rpy">

File: ika_robot_description/urdf/robot_base.xacro (robot description, xacro)
@@ -1,4 +1,5 @@
 <?xml version="1.0"?>
 <robot xmlns:xacro="http://www.ros.org/wiki/xacro">
+    <xacro:arg name="enable_traction" default="true"/>
     <xacro:property name="base_length" value="1.2"/>
     <xacro:property name="base_width" value="0.7"/>
@@ -10,4 +11,10 @@
     <xacro:property name="wheel_number" value="5"/>
     <xacro:property name="base_to_ground" value="${2*wheel_radius}"/>
+    <xacro:if value="$(arg enable_traction)">
+        <xacro:property name="front_radius" value="0.2"/>
+    </xacro:if>
+    <xacro:unless value="$(arg enable_traction)">
+        <xacro:property name="front_radius" value="0.3"/>
+    </xacro:unless>
     <link name="base_footprint"/>
     <joint name="base_joint" type="fixed">
@@ -35,19 +42,19 @@
     </link>
     <!-- Left Wheels -->
-    <xacro:macro name="left_wheel" params="id">
+    <xacro:macro name="left_wheel" params="id radii">
         <link name="left_wheel_${id}">
             <visual>
                 <geometry>
-                    <cylinder radius="${wheel_radius}" length="${wheel_length}"/>
+                    <cylinder radius="${radii}" length="${wheel_length}"/>
                 </geometry>
-                <material name="blue"/>
+                <material name="yellow"/>
             </visual>
             <collision>
                 <geometry>
-                    <sphere radius="${wheel_radius}"/>
-                    <!-- <cylinder radius="${wheel_radius}" length="${wheel_length}"/> -->
+                    <sphere radius="${radii}"/>
+                    <!-- <cylinder radius="${radii}" length="${wheel_length}"/> -->
                 </geometry>
             </collision>
-            <xacro:cylinder_inertia m="${wheel_mass}" r="${wheel_length}" l = "${wheel_length}"
+            <xacro:cylinder_inertia m="${wheel_mass}" r="${radii}" l = "${wheel_length}"
                                     xyz="0 0 0" rpy="0 0 0"/>
         </link>
@@ -60,25 +67,25 @@
         </joint>
     </xacro:macro>
-    <xacro:left_wheel id="1"/>
-    <xacro:left_wheel id="2"/>
-    <xacro:left_wheel id="3"/>
-    <xacro:left_wheel id="4"/>
-    <xacro:left_wheel id="5"/>
+    <xacro:left_wheel id="1" radii="${front_radius}"/>
+    <xacro:left_wheel id="2" radii="${wheel_radius}"/>
+    <xacro:left_wheel id="3" radii="${wheel_radius}"/>
+    <xacro:left_wheel id="4" radii="${wheel_radius}"/>
+    <xacro:left_wheel id="5" radii="${front_radius}"/>
     <!-- Right Wheels -->
-    <xacro:macro name="right_wheel" params="id">
+    <xacro:macro name="right_wheel" params="id radii">
         <link name="right_wheel_${id}">
             <visual>
                 <geometry>
-                    <cylinder radius="${wheel_radius}" length="${wheel_length}"/>
+                    <cylinder radius="${radii}" length="${wheel_length}"/>
                 </geometry>
-                <material name="blue" />
+                <material name="orange" />
             </visual>
             <collision>
                 <geometry>
-                    <sphere radius="${wheel_radius}"/>
-                    <!-- <cylinder radius="${wheel_radius}" length="${wheel_length}"/> -->
+                    <sphere radius="${radii}"/>
+                    <!-- <cylinder radius="${radii}" length="${wheel_length}"/> -->
                 </geometry>
             </collision>
-            <xacro:cylinder_inertia m="${wheel_mass}" r="${wheel_length}" l = "${wheel_length}"
+            <xacro:cylinder_inertia m="${wheel_mass}" r="${radii}" l = "${wheel_length}"
                                     xyz="0 0 0" rpy="0 0 0"/>
         </link>
@@ -91,32 +98,48 @@
         </joint>
     </xacro:macro>
-    <xacro:right_wheel id="1"/>
-    <xacro:right_wheel id="2"/>
-    <xacro:right_wheel id="3"/>
-    <xacro:right_wheel id="4"/>
-    <xacro:right_wheel id="5"/>
-    <xacro:macro name="create_gazebo_mu_001_wheel_tag" params="link_name color">
+    <xacro:right_wheel id="1" radii="${front_radius}"/>
+    <xacro:right_wheel id="2" radii="${wheel_radius}"/>
+    <xacro:right_wheel id="3" radii="${wheel_radius}"/>
+    <xacro:right_wheel id="4" radii="${wheel_radius}"/>
+    <xacro:right_wheel id="5" radii="${front_radius}"/>
+    <xacro:macro name="create_gazebo_wheel_tag" params="link_name color">
         <gazebo reference="${link_name}">
             <material>Gazebo/${color}</material>
-            <mu1 value="0.001"></mu1>
-            <mu2 value="0.001"></mu2>
+            <mu1 value="1"></mu1>
+            <mu2 value="1"></mu2>
         </gazebo>
     </xacro:macro>
-    <xacro:macro name="create_gazebo_mu_05_wheel_tag" params="link_name color">
+    <xacro:macro name="create_gazebo_mu_wheel_tag" params="link_name color mu">
         <gazebo reference="${link_name}">
             <material>Gazebo/${color}</material>
-            <mu1 value="0.05"></mu1>
-            <mu2 value="0.05"></mu2>
+            <mu1 value="${mu}"></mu1>
+            <mu2 value="${mu}"></mu2>
         </gazebo>
     </xacro:macro>
-    <xacro:create_gazebo_mu_001_wheel_tag link_name="left_wheel_1" color="Yellow"/>
-    <xacro:create_gazebo_mu_001_wheel_tag link_name="right_wheel_1" color="Orange"/>
-    <xacro:create_gazebo_mu_05_wheel_tag link_name="left_wheel_2" color="Yellow"/>
-    <xacro:create_gazebo_mu_05_wheel_tag link_name="right_wheel_2" color="Orange"/>
-    <xacro:create_gazebo_mu_05_wheel_tag link_name="left_wheel_4" color="Yellow"/>
-    <xacro:create_gazebo_mu_05_wheel_tag link_name="right_wheel_4" color="Orange"/>
-    <xacro:create_gazebo_mu_001_wheel_tag link_name="left_wheel_5" color="Yellow"/>
-    <xacro:create_gazebo_mu_001_wheel_tag link_name="right_wheel_5" color="Orange"/>
-    <gazebo reference="left_wheel_3">
+    <xacro:if value="$(arg enable_traction)">
+        <xacro:create_gazebo_wheel_tag link_name="left_wheel_1" color="Yellow"/>
+        <xacro:create_gazebo_wheel_tag link_name="right_wheel_1" color="Orange"/>
+        <xacro:create_gazebo_wheel_tag link_name="left_wheel_2" color="Yellow"/>
+        <xacro:create_gazebo_wheel_tag link_name="right_wheel_2" color="Orange"/>
+        <xacro:create_gazebo_wheel_tag link_name="left_wheel_3" color="Yellow"/>
+        <xacro:create_gazebo_wheel_tag link_name="right_wheel_3" color="Orange"/>
+        <xacro:create_gazebo_wheel_tag link_name="left_wheel_4" color="Yellow"/>
+        <xacro:create_gazebo_wheel_tag link_name="right_wheel_4" color="Orange"/>
+        <xacro:create_gazebo_wheel_tag link_name="left_wheel_5" color="Yellow"/>
+        <xacro:create_gazebo_wheel_tag link_name="right_wheel_5" color="Orange"/>
+    </xacro:if>
+    <xacro:unless value="$(arg enable_traction)">
+        <xacro:create_gazebo_mu_wheel_tag link_name="left_wheel_1"  color="Yellow" mu="0.001"/>
+        <xacro:create_gazebo_mu_wheel_tag link_name="right_wheel_1" color="Orange" mu="0.001"/>
+        <xacro:create_gazebo_mu_wheel_tag link_name="left_wheel_2"  color="Yellow" mu="0.05"/>
+        <xacro:create_gazebo_mu_wheel_tag link_name="right_wheel_2" color="Orange" mu="0.05"/>
+        <xacro:create_gazebo_wheel_tag    link_name="left_wheel_3"  color="Yellow"   />
+        <xacro:create_gazebo_wheel_tag    link_name="right_wheel_3" color="Orange"   />
+        <xacro:create_gazebo_mu_wheel_tag link_name="left_wheel_4"  color="Yellow" mu="0.05"/>
+        <xacro:create_gazebo_mu_wheel_tag link_name="right_wheel_4" color="Orange" mu="0.05"/>
+        <xacro:create_gazebo_mu_wheel_tag link_name="left_wheel_5"  color="Yellow" mu="0.001"/>
+        <xacro:create_gazebo_mu_wheel_tag link_name="right_wheel_5" color="Orange" mu="0.001"/>
+    </xacro:unless>
+    <!-- <gazebo reference="left_wheel_3">
         <material>Gazebo/Yellow</material>
         <mu1 value="1"></mu1>
@@ -127,4 +150,4 @@
         <mu1 value="1"></mu1>
         <mu2 value="1"></mu2>
-    </gazebo>
+    </gazebo> -->
 </robot>

File: ika_robot_description/urdf/ros2_control.xacro (robot description, xacro)
@@ -4,9 +4,10 @@
         <joint name="${prefix}">
             <command_interface name="velocity">
-                <param name="max">10</param>
-                <param name="min">-10</param>
+                <param name="max">100</param>
+                <param name="min">-100</param>
             </command_interface>
             <state_interface name="velocity"/>
             <state_interface name="position"/>
+            <param name="max_effort">100</param>
         </joint>
     </xacro:macro>

Commit message: added camera - depth camera - first barrier

File: ika_robot_description/urdf/common_properties.xacro (robot description, xacro)
@@ -15,4 +15,7 @@
     <material name="yellow">
         <color rgba="1 1 0 1"/>
+    </material>
+    <material name="red">
+        <color rgba="1 0 0 1"/>
     </material>
     <xacro:macro name="sphere_inertia" params="m r xyz rpy">

File: ika_robot_description/urdf/robot.xacro (robot description, xacro)
@@ -10,3 +10,5 @@
         <xacro:include filename="gazebo_control.xacro"/>
     </xacro:unless>
+    <!-- <xacro:include filename="camera.xacro"/> -->
+    <xacro:include filename="depth_camera.xacro"/>
 </robot>

File: ika_robot_description/urdf/robot_base.xacro (robot description, xacro)
@@ -1,4 +1,10 @@
 <?xml version="1.0"?>
 <robot xmlns:xacro="http://www.ros.org/wiki/xacro">
+    <!-- ADD WALLS -->
+    <!-- ADD CUSTOM MADE OBJECTS -->
+    <!-- USE DEPTH CAMERA -->
+    <!-- IMU -->
+    <!-- NAV2 WITH CAMERA -->
+    <!-- SECTION 5 -->
     <xacro:arg name="enable_traction" default="true"/>
     <xacro:property name="base_length" value="1.2"/>
