Commit message: robot_localization - nav2 - section5 done

File: ika_robot_description/urdf/depth_camera.xacro (robot description, xacro)
@@ -25,5 +25,5 @@
             <pose>0 0 0 0 0 0</pose>
             <visualize>true</visualize>
-            <update_rate>10.</update_rate>
+            <update_rate>20.</update_rate>
             <camera>
                 <horizontal_fov>1.52</horizontal_fov>

File: ika_robot_description/urdf/gazebo_control.xacro (robot description, xacro)
@@ -14,12 +14,14 @@
     </xacro:macro>
     <xacro:create_gazebo_wheel_tag link_name="base_link" color="Green"/>
-    <xacro:create_gazebo_caster_wheel_tag link_name="left_wheel_1" color="Orange"/>
+    <xacro:create_gazebo_caster_wheel_tag link_name="left_wheel_1" color="Yellow"/>
     <xacro:create_gazebo_caster_wheel_tag link_name="left_wheel_2" color="Yellow"/>
-    <xacro:create_gazebo_wheel_tag link_name="left_wheel_3" color="Orange"/>
+    <xacro:create_gazebo_wheel_tag link_name="left_wheel_3" color="Yellow"/>
     <xacro:create_gazebo_caster_wheel_tag link_name="left_wheel_4" color="Yellow"/>
-    <xacro:create_gazebo_caster_wheel_tag link_name="right_wheel_1" color="Yellow"/>
+    <xacro:create_gazebo_caster_wheel_tag link_name="left_wheel_5" color="Yellow"/>
+    <xacro:create_gazebo_caster_wheel_tag link_name="right_wheel_1" color="Orange"/>
     <xacro:create_gazebo_caster_wheel_tag link_name="right_wheel_2" color="Orange"/>
-    <xacro:create_gazebo_wheel_tag link_name="right_wheel_3" color="Yellow"/>
+    <xacro:create_gazebo_wheel_tag link_name="right_wheel_3" color="Orange"/>
     <xacro:create_gazebo_caster_wheel_tag link_name="right_wheel_4" color="Orange"/>
+    <xacro:create_gazebo_caster_wheel_tag link_name="right_wheel_5" color="Orange"/>
     <!-- GAZEBO DIFF DRIVE PLUGIN -->
     <xacro:macro name="create_diffdrive_cont" params="id">
@@ -54,4 +56,6 @@
             <joint_name>left_wheel_joint_4</joint_name>
             <joint_name>right_wheel_joint_4</joint_name>
+            <joint_name>left_wheel_joint_5</joint_name>
+            <joint_name>right_wheel_joint_5</joint_name>
             <update_rate>30.</update_rate>
         </plugin>

File: ika_robot_description/urdf/imu.xacro (robot description, xacro)
@@ -4,5 +4,5 @@
         <parent link="base_link"/>
         <child link="imu_link"/>
-        <origin xyz="0 0 ${base_hight}" rpy="0 0 0"/>
+        <origin xyz="0 0 ${base_hight/2}" rpy="0 0 0"/>
     </joint>
     <link name="imu_link"></link>

File: ika_robot_description/urdf/robot_base.xacro (robot description, xacro)
@@ -1,8 +1,4 @@
 <?xml version="1.0"?>
 <robot xmlns:xacro="http://www.ros.org/wiki/xacro">
-    <!-- ADD WALLS -->
-    <!-- ADD CUSTOM MADE OBJECTS -->
-    <!-- USE DEPTH CAMERA -->
-    <!-- IMU -->
     <!-- NAV2 WITH CAMERA -->
     <!-- SECTION 5 -->

Commit message: changed pointcloud and added the lighted world

File: ika_robot_description/urdf/depth_camera.xacro (robot description, xacro)
@@ -4,5 +4,5 @@
         <parent link="base_link"/>
         <child link="camera_link"/>
-        <origin xyz="${base_length/2 + 0.005} 0 ${base_hight/2}" rpy="0 0 0"/>
+        <origin xyz="${base_length/2 + 0.005} 0 ${base_hight+0.05}" rpy="0 0 0"/>
     </joint>
     <link name="camera_link">
@@ -29,5 +29,5 @@
                 <horizontal_fov>1.52</horizontal_fov>
                 <image>
-                    <format>B8R8G8</format>
+                    <format>BGR8</format>
                     <width>640</width>
                     <height>480</height>

File: ika_robot_description/urdf/robot.xacro (robot description, xacro)
@@ -11,6 +11,6 @@
     </xacro:unless>
     <!-- <xacro:include filename="camera.xacro"/> -->
-    <!-- <xacro:include filename="depth_camera.xacro"/> -->
-    <!-- <xacro:include filename="imu.xacro"/> -->
+    <xacro:include filename="depth_camera.xacro"/>
+    <xacro:include filename="imu.xacro"/>
     <!-- <xacro:include filename="laser_cam.xacro"/> -->
 </robot>

File: ika_robot_description/urdf/robot_base.xacro (robot description, xacro)
@@ -4,18 +4,19 @@
     <!-- SECTION 5 -->
     <xacro:arg name="enable_traction" default="true"/>
-    <xacro:property name="base_length" value="1.2"/>
-    <xacro:property name="base_width" value="0.7"/>
-    <xacro:property name="base_hight" value=".2"/>
-    <xacro:property name="base_mass" value="30."/>
-    <xacro:property name="wheel_radius" value="0.3"/>
-    <xacro:property name="wheel_length" value="0.3"/>
+    <xacro:property name="total_length" value="1.3"/>
+    <xacro:property name="base_length" value="1.218"/>
+    <xacro:property name="base_width" value="0.8"/>
+    <xacro:property name="base_hight" value=".37"/>
+    <xacro:property name="base_mass" value="40."/>
+    <xacro:property name="wheel_radius" value="0.26"/>
+    <xacro:property name="wheel_length" value="0.05"/>
     <xacro:property name="wheel_mass" value="5."/>
     <xacro:property name="wheel_number" value="5"/>
-    <xacro:property name="base_to_ground" value="${2*wheel_radius}"/>
+    <xacro:property name="base_to_ground" value="0.15"/>
     <xacro:if value="$(arg enable_traction)">
         <xacro:property name="front_radius" value="0.2"/>
     </xacro:if>
     <xacro:unless value="$(arg enable_traction)">
-        <xacro:property name="front_radius" value="0.3"/>
+        <xacro:property name="front_radius" value="0.26"/>
     </xacro:unless>
     <link name="base_footprint"/>
@@ -64,6 +65,6 @@
             <parent link="base_link"/>
             <child link="left_wheel_${id}"/>
-            <origin xyz="${base_length*(id-1)/(wheel_number-1) - base_length/2}
-                         ${base_width/2 + wheel_length/2} ${-wheel_radius}" rpy="${-pi/2.} 0 0"/>
+            <origin xyz="${(total_length-2*front_radius)*(id-1)/(wheel_number-1) - (total_length-2*front_radius)/2}
+                         ${base_width/2 + wheel_length/2} ${wheel_radius-base_to_ground}" rpy="${-pi/2.} 0 0"/>
             <axis xyz="0 0 1"/>
         </joint>
@@ -95,6 +96,6 @@
             <parent link="base_link"/>
             <child link="right_wheel_${id}"/>
-            <origin xyz="${base_length*(id-1)/(wheel_number-1) - base_length/2}
-                         -${base_width/2 + wheel_length/2} ${-wheel_radius}" rpy="${pi/2.} 0 0"/>
+            <origin xyz="${(total_length-2*front_radius)*(id-1)/(wheel_number-1) - (total_length-2*front_radius)/2}
+            -${base_width/2 + wheel_length/2} ${wheel_radius-base_to_ground}" rpy="${pi/2.} 0 0"/>
             <axis xyz="0 0 -1"/>
         </joint>
