Commit message: ff

File: ika_robot_description/urdf/lidar.xacro (robot description, xacro)
@@ -20,7 +20,6 @@
             </geometry>
         </collision>
-        <xacro:inertial_cylinder mass='0.1' length="${wheel_len}" radius="${wheel_rad}">
-            <origin xyz='0 0 0' rpy='0 0 0'/>
-        </xacro:inertial_cylinder>
+        <xacro:cylinder_inertia m="0.3" r="${wheel_rad}" l = "${wheel_len}"
+                                    xyz="0 0 0" rpy="0 0 0"/>
     </link>
     <gazebo reference='lidar_frame'>

File: ika_robot_description/urdf/robot.xacro (robot description, xacro)
@@ -13,5 +13,5 @@
     <!-- <xacro:include filename="depth_camera.xacro"/> -->
     <!-- <xacro:include filename="imu.xacro"/> -->
-    <!-- <xacro:include filename="lidar.xacro"/> -->
+    <xacro:include filename="lidar.xacro"/>
     <!-- <xacro:include filename="gps.xacro"/> -->
     <!-- <xacro:include filename="laser_cam.xacro"/> -->
